File: SuperPower-RPi-KiCAD/Pi-Batt.sch (KiCad schematic (older format))
At the start: 10 parts, among them J2 JST-PH, J4 DNP, Q1 Q_PMOS_DMP3056L-7_SOT-23, Q6 2N7002-7-F

Commit message: Final prep for distribution to KiCAD folks.
Other:
- note removed: "SSM3J328R"
Changed lines of the file:
@@
 encoding utf-8
 Sheet 5 8
-Title ""
-Date ""
-Rev ""
-Comp ""
-Comment1 ""
+Title "SuperPower-Leto"
+Date "2021-01-28"
+Rev "0.1"
+Comp "SuperPower Team"
+Comment1 "Drawn By: Seth Kazarians"
 Comment2 ""
 Comment3 ""
@@
 Wire Wire Line
 	4100 6250 4100 6000
-Text Notes 5600 2000 0    50   ~ 0
-SSM3J328R
 $Comp
 L Manual_Lib:Q_PMOS_DMP3056L-7_SOT-23 Q1
