File: SuperPower-RPi-KiCAD/Pi-Boost-Conv.sch (KiCad schematic (older format))
At the start: 26 parts, among them U1 TPS61088, U5 ME6210A33M3G

Commit message: Final prep for distribution to KiCAD folks.
Other:
- note removed: "Alternative component values:\nL1: 4.7uH\nC12: 39n\nR5: 169k\nR3: 412k"
- note removed: "NOTE:\nC12: Original design had 39nF. Changed to 47nF to reuse components.\nR4 & C13 values are taken from TPS61088 Eval Module schematic."
Changed lines of the file:
@@
 encoding utf-8
 Sheet 2 8
-Title ""
-Date ""
-Rev ""
-Comp ""
-Comment1 ""
+Title "SuperPower-Leto"
+Date "2021-01-28"
+Rev "0.1"
+Comp "SuperPower Team"
+Comment1 "Drawn By: Seth Kazarians"
 Comment2 ""
 Comment3 ""
@@
 	-1   0    0    1
 $EndComp
-Text Notes 750  7350 0    50   ~ 0
-Alternative component values:\nL1: 4.7uH\nC12: 39n\nR5: 169k\nR3: 412k
 Wire Wire Line
 	3050 1250 3150 1250
@@
 	1    0    0    -1
 $EndComp
-Text Notes 4500 5600 0    50   ~ 0
-NOTE:\nC12:  Original design had 39nF. Changed to 47nF to reuse components.\nR4 & C13 values are taken from TPS61088 Eval Module schematic.
 $EndSCHEMATC
