File: SuperPower-RPi-KiCAD/Pi-Charger.sch (KiCad schematic (older format))
At the start: 18 parts, among them U2 BQ25895RTW

Commit message: Final prep for distribution to KiCAD folks.
Other:
- note added: "NOTE:\nChanged footprint to use 0.3mm vias for BQ25895 and TPS61088"
- note removed: "Consider adding connection to ADC pin or device for ILIM"
- note removed: "NOTE:\nChange footprint to use 0.3mm vias for BQ25895 and TPS61088"
Changed lines of the file:
@@
 encoding utf-8
 Sheet 6 8
-Title ""
-Date ""
-Rev ""
-Comp ""
-Comment1 ""
+Title "SuperPower-Leto"
+Date "2021-01-28"
+Rev "0.1"
+Comp "SuperPower Team"
+Comment1 "Drawn By: Seth Kazarians"
 Comment2 ""
 Comment3 ""
@@
 $EndComp
 Text Notes 1200 6600 0    50   ~ 0
-NOTE:\nChange footprint to use 0.3mm vias for BQ25895 and TPS61088
+NOTE:\nChanged footprint to use 0.3mm vias for BQ25895 and TPS61088
 $Comp
 L Device:C_Small C26
@@
 Wire Wire Line
 	5050 4800 5050 4900
-Text Notes 1700 3750 0    50   ~ 0
-Consider adding connection to ADC pin or device for ILIM
 Text HLabel 4200 3550 0    50   Output ~ 0
 IMEAS
