File: SuperPower-RPi-KiCAD/Pi-Connection.sch (KiCad schematic (older format))
At the start: 1 part, among them J1 Raspberry_Pi_2_3

Commit message: Final prep for distribution to KiCAD folks.
Other:
- note removed: "Pins to STM32:\nGPIO5 to trigger update\nGPIO4 to indicate reboot/restart"
Changed lines of the file:
@@
 encoding utf-8
 Sheet 8 8
-Title ""
-Date ""
-Rev ""
-Comp ""
-Comment1 ""
+Title "SuperPower-Leto"
+Date "2021-01-28"
+Rev "0.1"
+Comp "SuperPower Team"
+Comment1 "Drawn By: Seth Kazarians"
 Comment2 ""
 Comment3 ""
@@
 NoConn ~ 5900 2300
 NoConn ~ 6000 2300
-Text Notes 1200 2500 0    50   ~ 0
-Pins to STM32:\nGPIO5 to trigger update\nGPIO4 to indicate reboot/restart
 Text HLabel 6800 3300 2    50   BiDi ~ 0
 GPIO4
