File: SuperPower-RPi-KiCAD/Pi-Input-Source.sch (KiCad schematic (older format))
At the start: 13 parts, among them J3 DNP, J6 USB_C_Receptacle_USB2.0, Q2 Q_PMOS_DMP3056L-7_SOT-23, Q3 Q_PMOS_DMP3056L-7_SOT-23, Q7 Q_PMOS_DMP3056L-7_SOT-23

Commit message: Final prep for distribution to KiCAD folks.
Other:
- note removed: "NOTE:\nscrew-terminals for solar."
Changed lines of the file:
@@
 encoding utf-8
 Sheet 4 8
-Title ""
-Date ""
-Rev ""
-Comp ""
-Comment1 ""
+Title "SuperPower-Leto"
+Date "2021-01-28"
+Rev "0.1"
+Comp "SuperPower Team"
+Comment1 "Drawn By: Seth Kazarians"
 Comment2 ""
 Comment3 ""
@@
 Text HLabel 9550 3000 2    50   Output ~ 0
 Vout
-Text Notes 1900 6400 0    50   ~ 0
-NOTE:\nscrew-terminals for solar.
 $Comp
 L Device:D_Zener_Small D3
