File: SuperPower-RPi-KiCAD/Pi-MCU.sch (KiCad schematic (older format))
At the start: 42 parts, among them J10 Conn_01x04, J11 QWIIC_Connector, J12 DNP, J13 Conn_01x06, J5 DNP, J7 Conn_01x03, J8 Conn_02x05_Odd_Even, J9 Conn_01x02, SW1 Tact, SW2 Tact, U3 STM32F412RETx, U4 ATtiny85-20SU

Commit message: Final prep for distribution to KiCAD folks.
Other:
- note removed: "I2C Pins: (SDA/SCL)\nI2C1: PB7/PB6 <--\nI2C2: PB3/PB10\nI2C3: PC9/PA8"
Changed lines of the file:
@@
 encoding utf-8
 Sheet 7 8
-Title ""
-Date ""
-Rev ""
-Comp ""
-Comment1 ""
+Title "SuperPower-Leto"
+Date "2021-01-28"
+Rev "0.1"
+Comp "SuperPower Team"
+Comment1 "Drawn By: Seth Kazarians"
 Comment2 ""
 Comment3 ""
@@
 Wire Wire Line
 	4200 4950 4250 4950
-Text Notes 3450 10700 0    50   ~ 0
-I2C Pins: (SDA/SCL)\nI2C1: PB7/PB6 <--\nI2C2: PB3/PB10\nI2C3: PC9/PA8
 Wire Wire Line
 	3050 7750 3450 7750
