File: SuperPower-RPi-KiCAD/SuperPower-RPi-KiCAD.kicad_pcb (KiCad board)
At the start: 2 copper layers, 65 x 56.5 mm, 122 parts, among them J1 Raspberry_Pi_2_3, J10 Conn_01x04, J11 QWIIC_Connector, J12 DNP, J13 Conn_01x06, J2 JST-PH, J3 DNP, J4 DNP, J5 DNP, J6 USB_C_Receptacle_USB2.0, J7 Conn_01x03, J8 Conn_02x05_Odd_Even, J9 Conn_01x02, Q1 Q_PMOS_DMP3056L-7_SOT-23, Q2 Q_PMOS_DMP3056L-7_SOT-23, Q3 Q_PMOS_DMP3056L-7_SOT-23, Q6 2N7002-7-F, Q7 Q_PMOS_DMP3056L-7_SOT-23, SW1 Tact, SW2 Tact, U1 TPS61088, U2 BQ25895RTW, U3 STM32F412RETx, U4 ATtiny85-20SU, U5 ME6210A33M3G, U6 NCP380HMU21AATBG

Commit message: Updated to KiCAD v5.99 (and undid the non-change)
Other:
- net class Default removed
